File: phantom-injector-hat.kicad_sch (KiCad schematic)
At the start: 41 parts, among them J1 Conn_02x20_Odd_Even, J2 Conn_02x03_Top_Bottom, J3 Conn_01x03, J4 Conn_01x03, SW1 SW_SPST, SW2 SW_SPST, U1 LT8362EMSE-PBF

Commit message: Fix all footprints; create initial PCB with board outline and DRU
Schematic footprint fixes (9 components had wrong or empty footprints):
- J1: empty → PinSocket_2x20_P2.54mm_Vertical (Pi GPIO stacking header)
- J2: empty → PinHeader_2x03_P2.54mm_Vertical (HiFiBerry J4 ribbon)
- J3/J4: SW_Slide_SPDT (wrong) → PinHeader_1x03_P2.54mm_Vertical (XLR pigtails)
- D1: D_SMB (wrong package) → D_SMA (B260A is DO-214AC/SMA)
- D2: empty → LED_D3.0mm (3mm through-hole LED)
- L2: empty → L_Wuerth_HCI-7040 (closest std footprint; verify pad layout)
- C3: SW_Slide_SPDT (wrong) → C_1206_3216Metric HandSolder
- C12: C_0805 (wrong size) → C_1812_4532Metric HandSolder

PCB:
- phantom-injector-hat.kicad_pcb: 65×56.5mm Pi HAT board outline from
  official KiCad template; 4× M2.5 mounting holes at spec positions;
  J1 GPIO header stripped (will be placed via Update PCB from Schematic
  at absolute pos 108.37,48.77 rot -90° per Pi HAT spec)
- phantom-injector-hat.kicad_dru: design rules (0.2mm signal, 0.5mm
  power, 0.5mm SW_NODE isolation, 0.3mm thermal via drill)
- Fixed empty group (id) parse error from template

Co-Authored-By: Claude Sonnet 4.6 <noreply@anthropic.com>
Parts:
- C12: footprint Capacitor_SMD:C_0805_2012Metric_Pad1.18x1.45mm_HandSolder -> Capacitor_SMD:C_1812_4532Metric_Pad1.57x3.40mm_HandSolder
- C3: footprint Button_Switch_THT:SW_Slide_SPDT_Angled_CK_OS102011MA1Q -> Capacitor_SMD:C_1206_3216Metric_Pad1.33x1.80mm_HandSolder
- D1: footprint Diode_SMD:D_SMB -> Diode_SMD:D_SMA
- D2: footprint (none) -> LED_THT:LED_D3.0mm
- J1: footprint (none) -> Connector_PinSocket_2.54mm:PinSocket_2x20_P2.54mm_Vertical
- J2: footprint (none) -> Connector_PinHeader_2.54mm:PinHeader_2x03_P2.54mm_Vertical
- J3, J4: footprint Button_Switch_THT:SW_Slide_SPDT_Angled_CK_OS102011MA1Q -> Connector_PinHeader_2.54mm:PinHeader_1x03_P2.54mm_Vertical
- L2: footprint (none) -> Inductor_SMD:L_Wuerth_HCI-7040
Changed lines of the file:
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@@
 	)
 	(label "GND"
-		(at 152.4 194.31 0)
+		(at 152.4 173.99 0)
 		(effects
 			(font
@@
 	)
 	(label "GND"
-		(at 152.4 163.83 0)
+		(at 139.7 189.23 180)
+		(effects
+			(font
+				(size 1.27 1.27)
+			)
+			(justify right bottom)
+		)
+	)
+	(label "GND"
+		(at 139.7 207.01 180)
+		(effects
+			(font
+				(size 1.27 1.27)
+			)
+			(justify right bottom)
+		)
+	)
+	(label "GND"
+		(at 152.4 181.61 0)
 		(effects
 			(font
@@
 	)
 	(label "GND"
-		(at 139.7 207.01 180)
-		(effects
-			(font
-				(size 1.27 1.27)
-			)
-			(justify right bottom)
-		)
-	)
-	(label "GND"
-		(at 152.4 173.99 0)
+		(at 152.4 194.31 0)
 		(effects
 			(font
@@
 	)
 	(label "GND"
-		(at 139.7 189.23 180)
+		(at 152.4 163.83 0)
 		(effects
 			(font
 				(size 1.27 1.27)
 			)
-			(justify right bottom)
+			(justify left bottom)
 		)
 	)
-	(label "GND"
-		(at 152.4 181.61 0)
+	(label "+5V_PI"
+		(at 152.4 158.75 0)
 		(effects
 			(font
@@
 		)
 	)
-	(label "+5V_PI"
-		(at 152.4 158.75 0)
-		(effects
-			(font
-				(size 1.27 1.27)
-			)
-			(justify left bottom)
-		)
-	)
 	(no_connect (at 45.72 185.42))
-	(no_connect (at 152.4 184.15))
-	(no_connect (at 152.4 191.77))
-	(no_connect (at 139.7 181.61))
 	(no_connect (at 139.7 158.75))
-	(no_connect (at 139.7 199.39))
-	(no_connect (at 139.7 201.93))
-	(no_connect (at 139.7 176.53))
-	(no_connect (at 139.7 161.29))
-	(no_connect (at 139.7 186.69))
+	(no_connect (at 139.7 166.37))
 	(no_connect (at 152.4 186.69))
 	(no_connect (at 139.7 194.31))
 	(no_connect (at 152.4 204.47))
-	(no_connect (at 152.4 166.37))
-	(no_connect (at 152.4 179.07))
-	(no_connect (at 152.4 189.23))
-	(no_connect (at 139.7 196.85))
-	(no_connect (at 152.4 176.53))
-	(no_connect (at 139.7 166.37))
-	(no_connect (at 139.7 163.83))
-	(no_connect (at 152.4 201.93))
-	(no_connect (at 139.7 171.45))
-	(no_connect (at 152.4 207.01))
-	(no_connect (at 139.7 204.47))
-	(no_connect (at 139.7 191.77))
+	(no_connect (at 139.7 181.61))
+	(no_connect (at 139.7 199.39))
 	(no_connect (at 152.4 196.85))
 	(no_connect (at 152.4 168.91))
+	(no_connect (at 139.7 171.45))
+	(no_connect (at 152.4 166.37))
+	(no_connect (at 152.4 191.77))
+	(no_connect (at 152.4 176.53))
+	(no_connect (at 139.7 196.85))
+	(no_connect (at 139.7 204.47))
+	(no_connect (at 139.7 173.99))
+	(no_connect (at 152.4 184.15))
+	(no_connect (at 152.4 189.23))
+	(no_connect (at 152.4 201.93))
+	(no_connect (at 139.7 176.53))
 	(no_connect (at 139.7 184.15))
+	(no_connect (at 152.4 207.01))
+	(no_connect (at 139.7 201.93))
+	(no_connect (at 139.7 163.83))
+	(no_connect (at 139.7 186.69))
 	(no_connect (at 139.7 179.07))
-	(no_connect (at 139.7 173.99))
+	(no_connect (at 139.7 191.77))
+	(no_connect (at 139.7 161.29))
+	(no_connect (at 152.4 179.07))
 	(no_connect (at 152.4 171.45))
 )

Commit message: Set SW1 and SW2 footprint to CK OS102011MA1Q slide switch
Co-Authored-By: Claude Sonnet 4.6 <noreply@anthropic.com>
Parts:
- SW1, SW2: footprint (none) -> Button_Switch_THT:SW_Slide_SPDT_Angled_CK_OS102011MA1Q
