File: phantom-injector-hat.kicad_pcb (KiCad board)
At the start: 2 copper layers, 65 x 56 mm, 45 parts, among them J1 Conn_02x20_Odd_Even, J2 Conn_02x03_Top_Bottom, J3 Conn_01x03, J4 Conn_01x03, SW1 SW_SPST, SW2 SW_SPST, U1 LT8362EMSE-PBF

Commit message: checkpoint
Parts:
- moved SW2 51.6 mm to (109.5, 77.0)
- moved SW1 51.5 mm to (109.5, 65.0)
- moved R6 30.5 mm to (119.0, 75.5), turned to 0 degrees
- moved R7 30.0 mm to (119.0, 79.0), turned to 0 degrees
- moved R9 28.7 mm to (122.5, 79.0), turned to 0 degrees
- moved R8 28.7 mm to (122.5, 75.5), turned to 0 degrees
- moved J3 25.8 mm to (156.2, 64.0)
- moved C14 24.7 mm to (120.5, 70.0), turned to 90 degrees
- moved J4 23.3 mm to (156.2, 73.5)
- moved MH3 18.0 mm to (103.5, 78.5)
- moved MH4 18.0 mm to (161.5, 78.5)
- moved C15 16.5 mm to (127.0, 77.0), turned to 90 degrees
- moved J2 16.3 mm to (143.0, 75.0), turned to 0 degrees
- moved C16 15.4 mm to (136.0, 77.0), turned to 90 degrees
- moved C13 12.5 mm to (127.0, 70.0), turned to 90 degrees
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Routing:
- net /+48V: track 58.6 -> 0.00 mm
- net /+5V_FILT: track 30.4 -> 0.00 mm
- net /+48V_RAW: track 25.1 -> 0.00 mm
- net /+5V_PI: track 22.0 -> 0.00 mm
- net /J4_L-: track 16.6 -> 0.00 mm
- net /J4_R-: track 16.5 -> 0.00 mm
- net /+48V_L: track 15.4 -> 0.00 mm
- net /+48V_R: track 14.0 -> 0.00 mm
- net /XLR_R_HOT: track 13.8 -> 0.00 mm
- net /XLR_L_HOT: track 13.6 -> 0.00 mm
- net /FBX: track 12.5 -> 0.00 mm
- net /XLR_R_COLD: track 12.4 -> 0.00 mm
- net /SW_NODE: track 10.6 -> 0.00 mm
- net /XLR_L_COLD: track 7.74 -> 0.00 mm
- net /J4_L+: track 6.21 -> 0.00 mm
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
Commit message: checkpoint before final layout and wiring
Parts:
- removed SW2: SW_SPST, Button_Switch_THT:SW_Slide_SPDT_Angled_CK_OS102011MA1Q
- FB1: footprint Inductor_SMD:L_1206_3216Metric_Pad1.22x1.90mm_HandSolder -> Inductor_SMD:L_0805_2012Metric_Pad1.05x1.20mm_HandSolder
- moved SW1 6.00 mm to (109.5, 71.0)
Connections:
- R6 pad 1: /+48V_L -> /+48V_SW
- R7 pad 1: /+48V_L -> /+48V_SW
- R8 pad 1: /+48V_R -> /+48V_SW
- R9 pad 1: /+48V_R -> /+48V_SW
- SW1 pad 2: /+48V_L -> /+48V_SW

Commit message: Starting routing and component layout
Parts:
- moved C8 10.9 mm to (108.5, 53.1), turned to -90 degrees
- moved C6 9.71 mm to (105.6, 53.1), turned to -90 degrees
- moved L2 7.94 mm to (115.0, 54.8)
Routing:
- net /+5V_PI: track 0.00 -> 6.97 mm
Changed lines of the file:
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@@
 	(footprint "Capacitor_SMD:C_0805_2012Metric_Pad1.18x1.45mm_HandSolder"
 		(layer "F.Cu")
-		(at 113.5 62.79 180)
+		(at 108.4836 53.0901 -90)
 		(descr "Capacitor SMD 0805 (2012 Metric), square (rectangular) end terminal, IPC-7351 nominal with elongated pad for handsoldering. (Body size source: IPC-SM-782 page 76, https://www.pcb-3d.com/wordpress/wp-content/uploads/ipc-sm-782a_amendment_1_and_2.pdf, https://docs.google.com/spreadsheets/d/1BsfQQcO9C6DZCsRaXUlFlo91Tg2WpOkGARC1WS5S8t0/edit?usp=sharing)")
 		(tags "capacitor handsolder")
 		(property "Reference" "C8"
-			(at 0 -1.68 0)
+			(at 2.6631 0.0508 180)
 			(layer "F.SilkS")
 			(effects
@@
 		)
 		(property "Value" "4.7 µF / 50V X7R"
-			(at 0 1.68 0)
+			(at 0 1.68 90)
 			(layer "F.Fab")
 			(effects
@@
 		)
 		(property "Datasheet" ""
-			(at 0 0 0)
+			(at 0 0 90)
 			(layer "F.Fab")
 			(hide yes)
@@
 		)
 		(property "Description" "Input EMI filter"
-			(at 0 0 0)
+			(at 0 0 90)
 			(layer "F.Fab")
 			(hide yes)
@@
 		)
 		(property "KiLib_Generator" "SMD_2terminal_chip_molded"
-			(at 0 0 0)
+			(at 0 0 90)
 			(layer "F.SilkS")
 			(hide yes)
@@
 		)
 		(fp_text user "${REFERENCE}"
-			(at 0 0 0)
+			(at 0 0 90)
 			(layer "F.Fab")
 			(effects
@@
 		)
 		(pad "1" smd roundrect
-			(at -1.0375 0 180)
+			(at -1.0375 0 270)
 			(size 1.175 1.45)
 			(layers "F.Cu" "F.Mask" "F.Paste")
@@
 		)
 		(pad "2" smd roundrect
-			(at 1.0375 0 180)
+			(at 1.0375 0 270)
 			(size 1.175 1.45)
 			(layers "F.Cu" "F.Mask" "F.Paste")
@@
 	(footprint "Capacitor_SMD:C_0805_2012Metric_Pad1.18x1.45mm_HandSolder"
 		(layer "F.Cu")
-		(at 113.5 58.73 180)
+		(at 105.592 53.0901 -90)
 		(descr "Capacitor SMD 0805 (2012 Metric), square (rectangular) end terminal, IPC-7351 nominal with elongated pad for handsoldering. (Body size source: IPC-SM-782 page 76, https://www.pcb-3d.com/wordpress/wp-content/uploads/ipc-sm-782a_amendment_1_and_2.pdf, https://docs.google.com/spreadsheets/d/1BsfQQcO9C6DZCsRaXUlFlo91Tg2WpOkGARC1WS5S8t0/edit?usp=sharing)")
 		(tags "capacitor handsolder")
 		(property "Reference" "C6"
-			(at 0 -1.68 0)
+			(at 2.7139 0.004 180)
 			(layer "F.SilkS")
 			(effects
@@
 		)
 		(property "Value" "22 µF / 16V X7R"
-			(at 0 1.68 0)
+			(at 0 1.68 90)
 			(layer "F.Fab")
 			(effects
@@
 		)
 		(property "Datasheet" ""
-			(at 0 0 0)
+			(at 0 0 90)
 			(layer "F.Fab")
 			(hide yes)
@@
 		)
 		(property "Description" "Bulk input"
-			(at 0 0 0)
+			(at 0 0 90)
 			(layer "F.Fab")
 			(hide yes)
@@
 		)
 		(property "KiLib_Generator" "SMD_2terminal_chip_molded"
-			(at 0 0 0)
+			(at 0 0 90)
 			(layer "F.SilkS")
 			(hide yes)
@@
 		)
 		(fp_text user "${REFERENCE}"
-			(at 0 0 0)
+			(at 0 0 90)
 			(layer "F.Fab")
 			(effects
@@
 		)
 		(pad "1" smd roundrect
-			(at -1.0375 0 180)
+			(at -1.0375 0 270)
 			(size 1.175 1.45)
 			(layers "F.Cu" "F.Mask" "F.Paste")
@@
 		)
 		(pad "2" smd roundrect
-			(at 1.0375 0 180)
+			(at 1.0375 0 270)
 			(size 1.175 1.45)
 			(layers "F.Cu" "F.Mask" "F.Paste")
@@
 	(footprint "Inductor_SMD:L_Wuerth_HCI-7040"
 		(layer "F.Cu")
-		(at 120 61)
+		(at 114.996 54.8388)
 		(descr "Inductor, Wuerth, HCI-7040, 6.9x6.9x3.8mm, (https://www.we-online.com/components/products/datasheet/744311022.pdf)")
 		(tags "flat-wire shielded Würth SMT")
@@
 		)
 	)
+	(segment
+		(start 105.592 49.008)
+		(end 105.592 52.0526)
+		(width 1)
+		(layer "F.Cu")
+		(net "/+5V_PI")
+	)
+	(segment
+		(start 108.37 46.23)
+		(end 105.592 49.008)
+		(width 1)
+		(layer "F.Cu")
+		(net "/+5V_PI")
+	)
 	(zone

Commit message: checkpointing layout and tracing
Parts:
- removed MH3, MH4: MountingHole_2.7mm_M2.5, MountingHole:MountingHole_2.7mm_M2.5
- moved C13 26.6 mm to (148.0, 86.4)
- moved C14 26.6 mm to (141.5, 86.4)
- moved C4 10.6 mm to (122.8, 67.2), turned to 180 degrees
- moved C9 8.39 mm to (141.8, 53.3)
- moved D1 7.93 mm to (136.4, 54.9)
- moved L1 7.12 mm to (129.6, 54.9)
- moved C18 6.91 mm to (121.5, 60.9), turned to -90 degrees
- moved R5 6.60 mm to (124.3, 55.9), turned to 90 degrees
- moved C1 5.62 mm to (121.5, 55.9), turned to -90 degrees
- moved SW1 5.04 mm to (111.3, 66.3), turned to -90 degrees
- moved R4 4.70 mm to (127.2, 67.2), turned to 180 degrees
- moved C2 4.31 mm to (127.2, 64.6), turned to 180 degrees
- moved U1 3.00 mm to (132.3, 60.8)
- moved C17 0.51 mm to (127.2, 61.9)
Routing:
- net /+5V_FILT: track 0.00 -> 28.9 mm
- net /+5V_PI: track 6.97 -> 17.5 mm
- net /SW_NODE: track 0.00 -> 8.31 mm
- net /EN_UVLO: track 0.00 -> 6.77 mm
- net /VC: track 0.00 -> 5.48 mm
- net /SYNC_MODE: track 0.00 -> 5.19 mm
- net /VC_COMP: track 0.00 -> 2.40 mm
- net /INTVCC: track 0.00 -> 2.31 mm
Other:
- board size 65 x 56 mm -> 65 x 40 mm

Commit message: Checkpoint routing
Parts:
- moved SW1 48.4 mm to (159.0, 58.5), turned to 90 degrees
- moved J2 30.4 mm to (114.1, 84.6), turned to 90 degrees
- moved C16 26.3 mm to (110.2, 82.0), turned to 0 degrees
- moved C13 24.9 mm to (123.1, 84.6), turned to 180 degrees
- moved C14 18.9 mm to (123.1, 82.0), turned to 180 degrees
- moved R8 18.6 mm to (106.3, 84.6)
- moved C15 18.4 mm to (110.2, 84.6), turned to 0 degrees
- moved R9 16.5 mm to (106.3, 82.0)
- moved R6 12.1 mm to (127.0, 84.6), turned to 180 degrees
- moved R7 8.59 mm to (127.0, 82.0), turned to 180 degrees
- moved D2 7.31 mm to (153.7, 54.5), turned to 90 degrees
- moved R10 2.52 mm to (153.7, 57.9), turned to 90 degrees
Routing:
- net /+48V_RAW: track 0.02 -> 14.5 mm
- net /+48V: track 0.00 -> 5.44 mm
- net /LED_A: track 0.00 -> 2.34 mm
Other:
- board size 65 x 40 mm -> 65 x 43.9 mm

Commit message: checkpoint all routed and layed out
Parts:
- moved SW1 53.0 mm to (107.1, 69.1), turned to -90 degrees
- moved J4 51.7 mm to (106.3, 87.1), turned to 180 degrees
- moved D2 49.5 mm to (104.8, 62.0), turned to 180 degrees
- moved R10 45.8 mm to (108.1, 62.0), turned to 180 degrees
- moved J3 37.3 mm to (127.0, 87.1), turned to 180 degrees
- moved FB1 13.4 mm to (146.7, 74.3)
- moved R1 8.31 mm to (131.1, 72.1)
- moved R2 8.31 mm to (128.0, 72.1)
- moved C12 8.31 mm to (134.4, 72.1)
- moved C10 5.90 mm to (146.7, 68.1)
- moved C11 5.90 mm to (146.7, 71.3)
- moved C3 5.90 mm to (146.7, 61.8)
- moved C7 5.90 mm to (146.7, 65.0)
- moved R8 3.80 mm to (102.5, 84.6)
- moved R9 3.80 mm to (102.5, 82.0)
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Routing:
- net /+48V: track 5.44 -> 63.5 mm
- net /+48V_SW: track 0.00 -> 47.5 mm
- net /+48V_RAW: track 14.5 -> 37.7 mm
- net /FBX: track 0.00 -> 14.9 mm
- net /RT: track 0.00 -> 8.06 mm
- net /SS: track 0.00 -> 6.05 mm
- net /XLR_R_HOT: track 0.00 -> 5.69 mm
- net /XLR_R_COLD: track 0.00 -> 5.69 mm
- net /XLR_L_HOT: track 0.00 -> 5.67 mm
- net /XLR_L_COLD: track 0.00 -> 5.67 mm
- net /J4_R-: track 0.00 -> 2.85 mm
- net /J4_R+: track 0.00 -> 2.85 mm
- net /J4_L-: track 0.00 -> 2.85 mm
- net /J4_L+: track 0.00 -> 2.85 mm
- net /LED_A: track 2.34 -> 0.00 mm
Other:
- board size 65 x 43.9 mm -> 65 x 44.8 mm
- board text removed: "DISPLAY (OPTIONAL)"
- board text removed: "PoE"

Commit message: mostly DRC clean
Routing:
- net /+48V_SW: track 47.5 -> 48.2 mm
Changed lines of the file:
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@@
+	)
+	(segment
+		(start 146.120292 75.3232)
+		(end 146.245292 75.1982)
+		(width 0.5)
+		(layer "F.Cu")
+		(net "/+48V")
 	)
 	(segment
@@
 		(start 147.8567 74.2932)
 		(end 147.8567 71.4309)
+		(width 0.5)
+		(layer "F.Cu")
+		(net "/+48V")
+	)
+	(segment
+		(start 109.3472 69.1308)
+		(end 121.0992 69.1308)
 		(width 0.5)
 		(layer "F.Cu")
@@
 	)
 	(segment
+		(start 144.868108 75.1982)
+		(end 144.993108 75.3232)
+		(width 0.5)
+		(layer "F.Cu")
+		(net "/+48V")
+	)
+	(segment
 		(start 147.8567 71.4309)
 		(end 147.7442 71.3184)
@@
 	)
 	(segment
-		(start 109.3472 69.1308)
-		(end 119.699688 69.1308)
-		(width 0.5)
-		(layer "F.Cu")
-		(net "/+48V")
-	)
-	(segment
-		(start 119.699688 69.1308)
-		(end 125.767088 75.1982)
-		(width 0.5)
-		(layer "F.Cu")
-		(net "/+48V")
-	)
-	(segment
 		(start 147.7442 71.3184)
 		(end 147.7442 68.1484)
@@
 	)
 	(segment
-		(start 125.767088 75.1982)
+		(start 146.245292 75.1982)
 		(end 146.9517 75.1982)
+		(width 0.5)
+		(layer "F.Cu")
+		(net "/+48V")
+	)
+	(segment
+		(start 127.1666 75.1982)
+		(end 144.868108 75.1982)
+		(width 0.5)
+		(layer "F.Cu")
+		(net "/+48V")
+	)
+	(segment
+		(start 121.0992 69.1308)
+		(end 127.1666 75.1982)
+		(width 0.5)
+		(layer "F.Cu")
+		(net "/+48V")
+	)
+	(segment
+		(start 144.993108 75.3232)
+		(end 146.120292 75.3232)
 		(width 0.5)
 		(layer "F.Cu")
@@
 	)
 	(segment
-		(start 107.112 71.1308)
-		(end 101.5052 76.7376)
+		(start 105.9584 71.1308)
+		(end 101.5052 75.584)
 		(width 0.5)
 		(layer "F.Cu")
@@
 	)
 	(segment
-		(start 101.5052 76.7376)
+		(start 101.5052 75.584)
 		(end 101.5052 82.0168)
 		(width 0.5)
 		(layer "F.Cu")
+		(net "/+48V_SW")
+	)
+	(segment
+		(start 107.112 71.1308)
+		(end 105.9584 71.1308)
+		(width 0.5)
+		(layer "F.Cu")

Commit message: Checkpoint
Routing:
- net /LED_A: track 0.00 -> 2.34 mm
Changed lines of the file:
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@@
 		(tags "Through hole pin header THT 1x03 2.54mm single row")
 		(property "Reference" "J3"
-			(at 0 -2.38 0)
+			(at 0 7.4676 0)
 			(layer "F.SilkS")
 			(effects
@@
 		(tags "Through hole pin header THT 1x03 2.54mm single row")
 		(property "Reference" "J4"
-			(at 0 -2.38 0)
+			(at 0 7.4676 0)
 			(layer "F.SilkS")
 			(effects
@@
 		(start 131.0916 73.06)
 		(end 134.3541 73.06)
-		(width 0.25)
+		(width 0.5)
 		(layer "F.Cu")
 		(net "/+48V_RAW")
@@
 		(start 134.3541 73.06)
 		(end 134.3916 73.0975)
-		(width 0.25)
+		(width 0.5)
 		(layer "F.Cu")
 		(net "/+48V_RAW")
@@
 	)
 	(segment
+		(start 104.7752 61.9508)
+		(end 107.112 61.9508)
+		(width 0.25)
+		(layer "F.Cu")
+		(net "/LED_A")
+	)
+	(segment
