File: phantom-injector-hat.kicad_pcb (KiCad board)
At the start: 2 copper layers, 65 x 44.8 mm, 42 parts, among them J1 Conn_02x20_Odd_Even, J2 Conn_02x03_Top_Bottom, J3 Conn_01x03, J4 Conn_01x03, SW1 SW_SPST, U1 LT8362EMSE-PBF

Commit message: WIP
Parts:
- moved FB1 8.96 mm to (144.9, 79.3), turned to 0 degrees
- moved R1 6.79 mm to (147.1, 76.9), turned to 0 degrees
- moved C12 3.20 mm to (147.0, 74.8), turned to 0 degrees
- moved C11 2.69 mm to (125.1, 70.2)
- moved R2 2.19 mm to (147.0, 72.6), turned to 180 degrees
- moved C10 1.81 mm to (122.9, 70.2)
- moved C7 0.91 mm to (120.6, 70.2)
Routing:
- net /+48V: track 33.7 -> 40.9 mm
- net /+48V_RAW: track 27.2 -> 21.0 mm
- net /FBX: track 10.3 -> 8.50 mm

Commit message: WIP
Parts:
- moved FB1 19.4 mm to (128.4, 69.1)
- moved C1 6.56 mm to (155.6, 65.5), turned to 90 degrees
- moved C18 5.76 mm to (153.5, 65.5), turned to 90 degrees
- moved C4 2.46 mm to (146.5, 63.3)
- moved C2 2.29 mm to (148.8, 67.3)
- moved R5 2.18 mm to (160.7, 63.4), turned to 180 degrees
- moved R4 2.11 mm to (146.5, 67.4)
- moved C17 1.57 mm to (151.2, 65.4)
- moved C9 0.36 mm to (160.1, 80.9)
- moved D1 0.36 mm to (160.1, 74.6)
- moved L1 0.36 mm to (160.1, 67.8)
Routing:
- net /+48V: track 40.9 -> 20.1 mm
- net /+48V_RAW: track 21.0 -> 40.1 mm
- net /+5V_FILT: track 65.7 -> 58.3 mm
- net /EN_UVLO: track 6.77 -> 12.6 mm
- net /INTVCC: track 2.31 -> 3.69 mm

Commit message: WIP
Parts:
- moved R1 8.40 mm to (154.3, 81.1), turned to 90 degrees
- moved C12 8.21 mm to (152.2, 81.1), turned to 90 degrees
- moved R2 7.71 mm to (148.7, 80.1)
Routing:
- net /FBX: track 8.50 -> 13.8 mm
Changed lines of the file:
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@@
 	(footprint "Capacitor_SMD:C_0805_2012Metric_Pad1.18x1.45mm_HandSolder"
 		(layer "F.Cu")
-		(at 146.99 74.7524)
+		(at 152.1716 81.1239 90)
 		(descr "Capacitor SMD 0805 (2012 Metric), square (rectangular) end terminal, IPC-7351 nominal with elongated pad for handsoldering. (Body size source: IPC-SM-782 page 76, https://www.pcb-3d.com/wordpress/wp-content/uploads/ipc-sm-782a_amendment_1_and_2.pdf, https://docs.google.com/spreadsheets/d/1BsfQQcO9C6DZCsRaXUlFlo91Tg2WpOkGARC1WS5S8t0/edit?usp=sharing)")
 		(tags "capacitor handsolder")
 		(property "Reference" "C12"
-			(at -3.1496 -0.0508 0)
+			(at -2.4677 -0.0508 0)
 			(layer "F.SilkS")
 			(effects
@@
 		)
 		(property "Value" "4.7 pF C0G"
-			(at 0 1.68 0)
+			(at 0 1.68 90)
 			(layer "F.Fab")
 			(effects
@@
 		)
 		(property "Datasheet" ""
-			(at 0 0 0)
+			(at 0 0 90)
 			(layer "F.Fab")
 			(hide yes)
@@
 		)
 		(property "Description" "FBX feedforward"
-			(at 0 0 0)
+			(at 0 0 90)
 			(layer "F.Fab")
 			(hide yes)
@@
 		)
 		(property "KiLib_Generator" "SMD_2terminal_chip_molded"
-			(at 0 0 0)
+			(at 0 0 90)
 			(layer "F.SilkS")
 			(hide yes)
@@
 		)
 		(fp_text user "${REFERENCE}"
-			(at 0 0 0)
+			(at 0 0 90)
 			(layer "F.Fab")
 			(effects
@@
 		)
 		(pad "1" smd roundrect
-			(at -1.0375 0)
+			(at -1.0375 0 90)
 			(size 1.175 1.45)
 			(layers "F.Cu" "F.Mask" "F.Paste")
@@
 		)
 		(pad "2" smd roundrect
-			(at 1.0375 0)
+			(at 1.0375 0 90)
 			(size 1.175 1.45)
 			(layers "F.Cu" "F.Mask" "F.Paste")
@@
 	(footprint "Resistor_SMD:R_0805_2012Metric_Pad1.20x1.40mm_HandSolder"
 		(layer "F.Cu")
-		(at 146.99 72.568 180)
+		(at 148.7172 80.0864 180)
 		(descr "Resistor SMD 0805 (2012 Metric), square (rectangular) end terminal, IPC-7351 nominal with elongated pad for handsoldering. (Body size source: IPC-SM-782 page 72, https://www.pcb-3d.com/wordpress/wp-content/uploads/ipc-sm-782a_amendment_1_and_2.pdf)")
 		(tags "resistor handsolder")
@@
 	(footprint "Resistor_SMD:R_0805_2012Metric_Pad1.20x1.40mm_HandSolder"
 		(layer "F.Cu")
-		(at 147.0568 76.886)
+		(at 154.3052 81.1239 90)
 		(descr "Resistor SMD 0805 (2012 Metric), square (rectangular) end terminal, IPC-7351 nominal with elongated pad for handsoldering. (Body size source: IPC-SM-782 page 72, https://www.pcb-3d.com/wordpress/wp-content/uploads/ipc-sm-782a_amendment_1_and_2.pdf)")
 		(tags "resistor handsolder")
 		(property "Reference" "R1"
-			(at -2.7084 0 0)
+			(at -2.4677 0 0)
 			(layer "F.SilkS")
 			(effects
@@
 		)
 		(property "Value" "1 MΩ 1%"
-			(at 0 1.65 0)
+			(at 0 1.65 90)
 			(layer "F.Fab")
 			(effects
@@
 		)
 		(property "Datasheet" ""
-			(at 0 0 0)
+			(at 0 0 90)
 			(layer "F.Fab")
 			(hide yes)
@@
 		)
 		(property "Description" "FBX top divider"
-			(at 0 0 0)
+			(at 0 0 90)
 			(layer "F.Fab")
 			(hide yes)
@@
 		)
 		(property "KiLib_Generator" "SMD_2terminal_chip_molded"
-			(at 0 0 0)
+			(at 0 0 90)
 			(layer "F.SilkS")
 			(hide yes)
@@
 		)
 		(fp_text user "${REFERENCE}"
-			(at 0 0 0)
+			(at 0 0 90)
 			(layer "F.Fab")
 			(effects
@@
 		)
 		(pad "1" smd roundrect
-			(at -1 0)
+			(at -1 0 90)
 			(size 1.2 1.4)
 			(layers "F.Cu" "F.Mask" "F.Paste")
@@
 		)
 		(pad "2" smd roundrect
-			(at 1 0)
+			(at 1 0 90)
 			(size 1.2 1.4)
 			(layers "F.Cu" "F.Mask" "F.Paste")
@@
 	)
 	(segment
-		(start 145.9525 74.7524)
-		(end 135.2552 74.7524)
-		(width 1)
-		(layer "F.Cu")
-		(net "/+48V_RAW")
-	)
-	(segment
-		(start 146.0572 76.8864)
-		(end 146.0568 76.886)
-		(width 1)
-		(layer "F.Cu")
-		(net "/+48V_RAW")
-	)
-	(segment
-		(start 146.0568 74.8567)
-		(end 145.9525 74.7524)
+		(start 154.2677 82.1614)
+		(end 154.3052 82.1239)
 		(width 1)
 		(layer "F.Cu")
@@
 	)
 	(segment
-		(start 146.0572 79.2736)
-		(end 146.0572 76.8864)
+		(start 157.2969 82.1239)
+		(end 160.0964 79.3244)
 		(width 1)
 		(layer "F.Cu")
@@
 	)
 	(segment
-		(start 146.0572 79.2736)
-		(end 160.0456 79.2736)
+		(start 152.1716 82.1614)
+		(end 142.595 82.1614)
 		(width 1)
 		(layer "F.Cu")
@@
 	)
 	(segment
-		(start 146.108 79.3244)
-		(end 146.0572 79.2736)
+		(start 160.0964 76.6396)
+		(end 160.0964 79.3244)
 		(width 1)
 		(layer "F.Cu")
@@
 	)
 	(segment
-		(start 129.6164 69.1136)
+		(start 142.595 82.1614)
 		(end 129.5472 69.1136)
 		(width 1)
@@
 	)
 	(segment
-		(start 146.0568 76.886)
-		(end 146.0568 74.8567)
-		(width 1)
-		(layer "F.Cu")
-		(net "/+48V_RAW")
-	)
-	(segment
-		(start 160.0456 79.2736)
-		(end 160.0964 79.3244)
+		(start 154.3052 82.1239)
+		(end 157.2969 82.1239)
 		(width 1)
 		(layer "F.Cu")
@@
 	)
 	(segment
-		(start 160.0964 79.3244)
-		(end 160.0964 76.6396)
+		(start 152.1716 82.1614)
+		(end 154.2677 82.1614)
 		(width 1)
 		(layer "F.Cu")
@@
 	)
 	(segment
-		(start 135.2552 74.7524)
-		(end 129.6164 69.1136)
-		(width 1)
+		(start 152.2091 80.1239)
+		(end 152.1716 80.0864)
+		(width 0.25)
 		(layer "F.Cu")
-		(net "/+48V_RAW")
+		(net "/FBX")
 	)
 	(segment
-		(start 152.12337 72.6264)
-		(end 148.0484 72.6264)
+		(start 149.4394 74.384784)
+		(end 151.197784 72.6264)
 		(width 0.25)
 		(layer "F.Cu")
@@
 	)
 	(segment
-		(start 148.0275 76.8567)
-		(end 148.0568 76.886)
+		(start 149.4394 79.8086)
+		(end 149.4394 74.384784)
 		(width 0.25)
 		(layer "F.Cu")
@@
 	)
 	(segment
-		(start 147.99 72.568)
-		(end 147.99 74.7149)
+		(start 149.7172 80.0864)
+		(end 149.4394 79.8086)
 		(width 0.25)
 		(layer "F.Cu")
@@
 	)
 	(segment
-		(start 148.0484 72.6264)
-		(end 147.99 72.568)
+		(start 154.3052 80.1239)
+		(end 152.2091 80.1239)
 		(width 0.25)
 		(layer "F.Cu")
@@
 	)
 	(segment
-		(start 147.99 74.7149)
-		(end 148.0275 74.7524)
+		(start 151.197784 72.6264)
+		(end 152.12337 72.6264)
 		(width 0.25)
 		(layer "F.Cu")
@@
 	)
 	(segment
-		(start 148.0275 74.7524)
-		(end 148.0275 76.8567)
+		(start 152.1716 80.0864)
+		(end 149.7172 80.0864)
 		(width 0.25)
 		(layer "F.Cu")

Commit message: WIP
Parts:
- moved C10 27.3 mm to (147.8, 81.3)
- moved C11 27.3 mm to (150.1, 81.3)
- moved C7 27.3 mm to (145.5, 81.3)
- moved C3 27.3 mm to (143.2, 81.3)
- moved FB1 27.3 mm to (153.3, 80.2)
- moved R1 13.7 mm to (144.4, 71.6), turned to -90 degrees
- moved C12 11.1 mm to (146.6, 71.6), turned to -90 degrees
- moved R2 8.50 mm to (149.0, 71.6), turned to 90 degrees
- moved C9 1.63 mm to (158.5, 80.9)
- moved D1 1.63 mm to (158.5, 74.6)
- moved C5 1.01 mm to (152.1, 76.0)
- moved R11 1.01 mm to (154.8, 76.0)
- moved R3 1.01 mm to (149.4, 76.0)
- moved C4 0.97 mm to (146.5, 62.4)
- moved C2 0.97 mm to (148.8, 66.4)
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Routing:
- net /+48V: track 20.1 -> 49.7 mm
- net /+48V_RAW: track 39.8 -> 26.7 mm
- net /FBX: track 13.8 -> 7.72 mm
- net /SYNC_MODE: track 3.53 -> 2.39 mm
- net /RT: track 3.56 -> 4.58 mm
- net /SW_NODE: track 8.66 -> 7.71 mm
- net /SS: track 2.32 -> 3.16 mm

Commit message: Chkpt
Parts:
- moved R3 0.66 mm to (150.1, 76.0)
- moved C5 0.33 mm to (152.4, 76.0)
- moved C1 0.10 mm to (155.7, 65.5)
Routing:
- net /RT: track 4.58 -> 3.92 mm
- net /SS: track 3.16 -> 2.60 mm
Changed lines of the file:
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@@
 	(footprint "Capacitor_SMD:C_0805_2012Metric_Pad1.18x1.45mm_HandSolder"
 		(layer "F.Cu")
-		(at 152.0924 75.9716 -90)
+		(at 152.4256 75.9716 -90)
 		(descr "Capacitor SMD 0805 (2012 Metric), square (rectangular) end terminal, IPC-7351 nominal with elongated pad for handsoldering. (Body size source: IPC-SM-782 page 76, https://www.pcb-3d.com/wordpress/wp-content/uploads/ipc-sm-782a_amendment_1_and_2.pdf, https://docs.google.com/spreadsheets/d/1BsfQQcO9C6DZCsRaXUlFlo91Tg2WpOkGARC1WS5S8t0/edit?usp=sharing)")
 		(tags "capacitor handsolder")
@@
 	(footprint "Resistor_SMD:R_0805_2012Metric_Pad1.20x1.40mm_HandSolder"
 		(layer "F.Cu")
-		(at 149.4324 75.9716 -90)
+		(at 150.0888 75.9716 -90)
 		(descr "Resistor SMD 0805 (2012 Metric), square (rectangular) end terminal, IPC-7351 nominal with elongated pad for handsoldering. (Body size source: IPC-SM-782 page 72, https://www.pcb-3d.com/wordpress/wp-content/uploads/ipc-sm-782a_amendment_1_and_2.pdf)")
 		(tags "resistor handsolder")
@@
 	(footprint "Capacitor_SMD:C_0805_2012Metric_Pad1.18x1.45mm_HandSolder"
 		(layer "F.Cu")
-		(at 155.626 65.4853 90)
+		(at 155.7276 65.4853 90)
 		(descr "Capacitor SMD 0805 (2012 Metric), square (rectangular) end terminal, IPC-7351 nominal with elongated pad for handsoldering. (Body size source: IPC-SM-782 page 76, https://www.pcb-3d.com/wordpress/wp-content/uploads/ipc-sm-782a_amendment_1_and_2.pdf, https://docs.google.com/spreadsheets/d/1BsfQQcO9C6DZCsRaXUlFlo91Tg2WpOkGARC1WS5S8t0/edit?usp=sharing)")
 		(tags "capacitor handsolder")
@@
 	)
 	(segment
-		(start 153.12413 74.62737)
-		(end 153.12413 72.6264)
+		(start 153.12413 72.6264)
+		(end 153.12413 74.23557)
 		(width 0.25)
 		(layer "F.Cu")
@@
 	)
 	(segment
-		(start 152.0924 74.9341)
-		(end 152.8174 74.9341)
-		(width 0.25)
-		(layer "F.Cu")
-		(net "/SS")
-	)
-	(segment
-		(start 152.8174 74.9341)
-		(end 153.12413 74.62737)
+		(start 153.12413 74.23557)
+		(end 152.4256 74.9341)
 		(width 0.25)
 		(layer "F.Cu")
@@
 	)
 	(segment
-		(start 154.7624 74.9716)
-		(end 154.7624 74.255555)
+		(start 153.62451 73.83371)
+		(end 154.7624 74.9716)
 		(width 0.25)
 		(layer "F.Cu")
@@
 	)
 	(segment
-		(start 154.7624 74.255555)
-		(end 153.58153 73.074685)
+		(start 153.62451 72.6264)
+		(end 153.62451 73.83371)
 		(width 0.25)
 		(layer "F.Cu")
@@
 	)
 	(segment
-		(start 152.62375 72.6264)
+		(start 152.06787 73.8888)
 		(end 152.62375 73.33292)
 		(width 0.25)
@@
 	)
 	(segment
-		(start 151.91507 74.0416)
-		(end 150.3624 74.0416)
+		(start 152.62375 73.33292)
+		(end 152.62375 72.6264)
 		(width 0.25)
 		(layer "F.Cu")
@@
 	)
 	(segment
-		(start 152.62375 73.33292)
-		(end 151.91507 74.0416)
+		(start 151.1716 73.8888)
+		(end 152.06787 73.8888)
 		(width 0.25)
 		(layer "F.Cu")
@@
 	)
 	(segment
-		(start 150.3624 74.0416)
-		(end 149.4324 74.9716)
+		(start 150.0888 74.9716)
+		(end 151.1716 73.8888)
 		(width 0.25)
 		(layer "F.Cu")
@@
 	)
 	(segment
-		(start 155.626 72.6264)
-		(end 154.62524 72.6264)
-		(width 1.5)
+		(start 154.62527 72.6264)
+		(end 155.626 72.6264)
+		(width 1.25)
 		(layer "F.Cu")
 		(net "/SW_NODE")

Commit message: CHKP
Parts:
- moved SW1 1.51 mm to (107.1, 67.6)
- moved C3 1.09 mm to (144.3, 81.3)
- moved FB1 1.09 mm to (154.4, 80.2)
- moved C10 1.09 mm to (148.9, 81.3)
- moved C11 1.09 mm to (151.2, 81.3)
- moved C7 1.09 mm to (146.6, 81.3)
- moved C5 0.61 mm to (153.0, 76.0)
- moved R11 0.61 mm to (155.4, 76.0)
- moved R3 0.61 mm to (150.7, 76.0)
Routing:
- net /+48V_SW: track 50.2 -> 53.3 mm
- net /+48V: track 49.7 -> 51.4 mm
- net /RT: track 3.92 -> 3.31 mm

Commit message: Checkpoint
Parts:
- moved SW1 37.1 mm to (140.5, 83.7), turned to 0 degrees
- moved D2 33.7 mm to (104.1, 73.2), turned to 180 degrees
- moved R10 26.3 mm to (107.5, 75.5), turned to 90 degrees
- moved L1 3.86 mm to (161.6, 64.2)
- moved R2 3.77 mm to (150.3, 68.1)
- moved C18 3.62 mm to (152.9, 61.9)
- moved C1 3.62 mm to (155.1, 61.9)
- moved C17 3.62 mm to (150.5, 61.9)
- moved C10 3.56 mm to (148.9, 77.7)
- moved C11 3.56 mm to (151.2, 77.7)
- moved C3 3.56 mm to (144.3, 77.7)
- moved C7 3.56 mm to (146.6, 77.7)
- moved D1 3.56 mm to (158.5, 71.1)
- moved C5 3.56 mm to (153.0, 72.4)
- moved C9 3.56 mm to (158.5, 77.3)
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Connections:
- SW1 pad 1: /+48V -> /+48V_SW
- SW1 pad 2: /+48V_SW -> /+48V
Routing:
- net /+48V: track 51.4 -> 17.1 mm
- net /EN_UVLO: track 12.6 -> 1.72 mm
- net /+48V_RAW: track 27.1 -> 19.4 mm
- net /+48V_SW: track 53.3 -> 57.3 mm
- net /+5V_FILT: track 58.3 -> 61.8 mm
- net /LED_A: track 5.44 -> 3.93 mm
- net /FBX: track 7.72 -> 6.26 mm
- net /SW_NODE: track 7.71 -> 8.32 mm
- net /INTVCC: track 3.69 -> 4.30 mm
