File: phantom-injector-hat.kicad_pcb (KiCad board)
At the start: 2 copper layers, 65 x 44.8 mm, 42 parts, among them J1 Conn_02x20_Odd_Even, J2 Conn_02x03_Top_Bottom, J3 Conn_01x03, J4 Conn_01x03, SW1 SW_SPST, U1 LT8362EMSE-PBF

Commit message: WIP
Other:
- board text removed: "Extend PCB edge 0.5mm if using SMT header"
Changed lines of the file:
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@@
 		(tags "resistor handsolder")
 		(property "Reference" "R2"
-			(at 1.1696 -1.646 180)
+			(at 1.068 -1.5444 180)
 			(layer "F.SilkS")
 			(effects
@@
 		(layer "Edge.Cuts")
 	)
-	(gr_text "Extend PCB edge 0.5mm if using SMT header"
-		(at 103 42.5 0)
-		(layer "Dwgs.User")
-		(effects
-			(font
-				(size 1 1)
-				(thickness 0.15)
-			)
-			(justify left)
-		)
-	)
 	(gr_text "RJ45"

Commit message: wip
Parts:
- moved FB1 9.10 mm to (147.6, 65.7)
- moved C11 9.07 mm to (148.6, 69.2)
- moved R1 9.07 mm to (141.0, 76.1)
- moved R3 9.05 mm to (143.3, 71.1)
- moved C10 9.05 mm to (148.6, 71.8)
- moved C12 9.05 mm to (141.0, 73.6)
- moved C4 9.05 mm to (128.4, 73.5)
- moved R4 9.05 mm to (132.5, 73.5)
- moved R11 9.05 mm to (143.3, 65.4)
- moved C7 9.04 mm to (148.6, 74.3)
- moved R2 9.04 mm to (139.0, 71.1)
- moved R5 9.04 mm to (134.5, 56.9)
- moved C17 9.04 mm to (135.7, 72.0)
- moved C2 9.03 mm to (132.4, 70.9)
- moved L1 9.03 mm to (135.1, 61.3)
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Routing:
- net /+48V_SW: track 66.0 -> 56.9 mm
- net /+5V_FILT: track 41.8 -> 33.2 mm
- net /+48V: track 14.0 -> 15.1 mm
- net /FBX: track 6.26 -> 7.05 mm
- net /SYNC_MODE: track 3.07 -> 3.70 mm
- net /RT: track 3.31 -> 3.94 mm
- net /+48V_RAW: track 21.3 -> 21.8 mm

Commit message: CHeckpoint
Routing:
- net /+5V_FILT: track 33.2 -> 32.4 mm
Changed lines of the file:
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@@
-	)
-	(segment
-		(start 138.1856 79.3912)
-		(end 137.9824 79.3912)
-		(width 1)
-		(layer "F.Cu")
-		(net "/+48V_SW")
 	)
 	(segment
@@
 	)
 	(segment
-		(start 147.5666 81.959)
-		(end 147.5736 81.966)
-		(width 1)
-		(layer "F.Cu")
-		(net "/+48V")
-	)
-	(segment
-		(start 147.5588 69.2087)
-		(end 147.5666 69.2165)
-		(width 1)
-		(layer "F.Cu")
-		(net "/+48V")
-	)
-	(segment
 		(start 133.44995 70.9218)
 		(end 133.91603 70.9218)
@@
 	)
 	(segment
-		(start 133.45245 70.9243)
-		(end 133.44995 70.9218)
-		(width 0.25)
-		(layer "F.Cu")
-		(net "/VC")
-	)
-	(segment
 		(start 147.5588 64.56)
 		(end 147.5588 61.5321)
@@
 	)
 	(segment
-		(start 141.956 73.6996)
-		(end 142.031 73.6246)
-		(width 0.5)
-		(layer "F.Cu")
-		(net "/+48V_RAW")
-	)
-	(segment
 		(start 146.0248 66.094)
 		(end 147.5588 64.56)
@@
 	)
 	(segment
-		(start 147.5588 61.5321)
-		(end 147.5203 61.4936)
-		(width 1)
-		(layer "F.Cu")
-		(net "/+48V_RAW")
-	)
-	(segment
 		(start 144.1554 73.6246)
 		(end 146.0248 71.7552)
@@
 	)
 	(segment
-		(start 139.9636 71.114)
-		(end 139.9748 71.1252)
-		(width 0.25)
-		(layer "F.Cu")
-		(net "/FBX")
-	)
-	(segment
 		(start 139.956 73.6246)
 		(end 139.956 76.124)
@@
 	)
 	(segment
-		(start 139.9748 73.6058)
-		(end 139.956 73.6246)
-		(width 0.25)
-		(layer "F.Cu")
-		(net "/FBX")
-	)
-	(segment
 		(start 139.9748 71.1252)
 		(end 139.9748 73.6058)
@@
 	)
 	(segment
-		(start 142.2713 68.25)
-		(end 142.11117 68.08987)
-		(width 0.25)
-		(layer "F.Cu")
-		(net "/SS")
-	)
-	(segment
 		(start 142.11117 68.08987)
 		(end 139.9636 68.08987)
@@
 	)
 	(segment
-		(start 119.9184 84.6584)
-		(end 119.9 84.64)
-		(width 1)
-		(layer "F.Cu")
-		(net "/J4_L+")
-	)
-	(segment
 		(start 122.7584 84.6584)
 		(end 119.9184 84.6584)
@@
 	)
 	(segment
-		(start 133.4579 66.1038)
-		(end 133.4657 66.096)
-		(width 1)
-		(layer "F.Cu")
-		(net "/+5V_FILT")
-	)
-	(segment
-		(start 133.4826 56.927)
-		(end 133.4772 56.9216)
-		(width 1)
-		(layer "F.Cu")
-		(net "/+5V_FILT")
-	)
-	(segment
-		(start 133.4657 61.4901)
-		(end 133.4826 61.4732)
-		(width 1)
-		(layer "F.Cu")
-		(net "/+5V_FILT")
-	)
-	(segment
 		(start 131.725 59.7156)
 		(end 133.4826 61.4732)
@@
 	)
 	(segment
-		(start 133.4579 68.3312)
-		(end 133.71695 68.59025)
-		(width 0.5)
-		(layer "F.Cu")
-		(net "/+5V_FILT")
-	)
-	(segment
-		(start 133.4826 61.4732)
-		(end 133.4826 61.0882)
-		(width 1)
-		(layer "F.Cu")
-		(net "/+5V_FILT")
-	)
-	(segment
 		(start 133.4657 66.096)
 		(end 133.4657 61.4901)
@@
 	)
 	(segment
-		(start 133.4826 61.0882)
-		(end 133.4772 61.0828)
-		(width 1)
-		(layer "F.Cu")
-		(net "/+5V_FILT")
-	)
-	(segment
 		(start 117.546 59.7156)
 		(end 131.725 59.7156)
@@
 	)
 	(segment
-		(start 111.99 84.64)
-		(end 111.9716 84.6584)
-		(width 1)
-		(layer "F.Cu")
-		(net "/J4_R-")
-	)
-	(segment
 		(start 114.82 84.64)
 		(end 111.99 84.64)
@@
 	)
 	(segment
-		(start 111.99 82.1)
-		(end 111.9716 82.1184)
-		(width 1)
-		(layer "F.Cu")
-		(net "/J4_R+")
-	)
-	(segment
 		(start 119.9 82.1)
 		(end 122.74 82.1)
@@
 	)
 	(segment
-		(start 122.74 82.1)
-		(end 122.7584 82.1184)
-		(width 1)
-		(layer "F.Cu")
-		(net "/J4_L-")
-	)
-	(segment
 		(start 142.3088 70.22893)
 		(end 140.67012 68.59025)
@@
 	)
 	(segment
-		(start 138.2016 81.4072)
-		(end 138.1856 81.3912)
-		(width 1)
-		(layer "F.Cu")
-		(net "/LED_A")
-	)
-	(segment
 		(start 138.2016 83.8456)
 		(end 138.2016 81.4072)
@@
 		(layer "F.Cu")
 		(net "/LED_A")
-	)
-	(segment
-		(start 139.9564 61.4732)
-		(end 139.9768 61.4936)
-		(width 1.5)
-		(layer "F.Cu")
-		(net "/SW_NODE")
-	)
-	(segment
-		(start 139.9636 61.5068)
-		(end 139.9768 61.4936)
-		(width 1.5)
-		(layer "F.Cu")
-		(net "/SW_NODE")
 	)
 	(segment
@@
 	)
 	(segment
-		(start 135.4772 56.9216)
-		(end 135.4176 56.9812)
-		(width 0.25)
-		(layer "F.Cu")
-		(net "/EN_UVLO")
-	)
-	(segment

Commit message: Checkpoint
Parts:
- moved C1 0.23 mm to (132.4, 65.9)
Routing:
- net /GND: vias 7 -> 45

Commit message: WIP
Parts:
- C6: footprint Capacitor_SMD:C_0805_2012Metric_Pad1.18x1.45mm_HandSolder -> Capacitor_SMD:C_1210_3225Metric_Pad1.33x2.70mm_HandSolder
- moved C6 0.52 mm to (106.2, 61.3)
- moved C8 0.21 mm to (109.3, 60.8)
Changed lines of the file:
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@@
 	(footprint "Capacitor_SMD:C_0805_2012Metric_Pad1.18x1.45mm_HandSolder"
 		(layer "F.Cu")
-		(at 109.14 60.7531 -90)
+		(at 109.3472 60.7531 -90)
 		(descr "Capacitor SMD 0805 (2012 Metric), square (rectangular) end terminal, IPC-7351 nominal with elongated pad for handsoldering. (Body size source: IPC-SM-782 page 76, https://www.pcb-3d.com/wordpress/wp-content/uploads/ipc-sm-782a_amendment_1_and_2.pdf, https://docs.google.com/spreadsheets/d/1BsfQQcO9C6DZCsRaXUlFlo91Tg2WpOkGARC1WS5S8t0/edit?usp=sharing)")
 		(tags "capacitor handsolder")
@@
 		(embedded_fonts no)
 	)
-	(footprint "Capacitor_SMD:C_0805_2012Metric_Pad1.18x1.45mm_HandSolder"
+	(footprint "Capacitor_SMD:C_1210_3225Metric_Pad1.33x2.70mm_HandSolder"
 		(layer "F.Cu")
-		(at 106.2484 60.7531 -90)
-		(descr "Capacitor SMD 0805 (2012 Metric), square (rectangular) end terminal, IPC-7351 nominal with elongated pad for handsoldering. (Body size source: IPC-SM-782 page 76, https://www.pcb-3d.com/wordpress/wp-content/uploads/ipc-sm-782a_amendment_1_and_2.pdf, https://docs.google.com/spreadsheets/d/1BsfQQcO9C6DZCsRaXUlFlo91Tg2WpOkGARC1WS5S8t0/edit?usp=sharing)")
+		(at 106.2484 61.2781 -90)
+		(descr "Capacitor SMD 1210 (3225 Metric), square (rectangular) end terminal, IPC-7351 nominal with elongated pad for handsoldering. (Body size source: IPC-SM-782 page 76, https://www.pcb-3d.com/wordpress/wp-content/uploads/ipc-sm-782a_amendment_1_and_2.pdf)")
 		(tags "capacitor handsolder")
 		(property "Reference" "C6"
-			(at 2.7139 0.004 180)
+			(at 3.3821 0.0508 0)
 			(layer "F.SilkS")
 			(effects
 				(font
-					(size 0.8 0.8)
+					(size 1 1)
 					(thickness 0.15)
 				)
@@
 		)
 		(property "Value" "22 µF / 16V X7R"
-			(at 0 1.68 90)
+			(at 0 2.3 270)
 			(layer "F.Fab")
 			(effects
@@
 		)
 		(property "Datasheet" ""
-			(at 0 0 90)
+			(at 0 0 270)
 			(layer "F.Fab")
 			(hide yes)
@@
 		)
 		(property "Description" "Bulk input"
-			(at 0 0 90)
+			(at 0 0 270)
 			(layer "F.Fab")
 			(hide yes)
@@
 		)
 		(property "KiLib_Generator" "SMD_2terminal_chip_molded"
-			(at 0 0 90)
+			(at 0 0 270)
 			(layer "F.SilkS")
 			(hide yes)
@@
 		(duplicate_pad_numbers_are_jumpers no)
 		(fp_line
-			(start -0.261252 0.735)
-			(end 0.261252 0.735)
+			(start -0.711252 1.36)
+			(end 0.711252 1.36)
 			(stroke
 				(width 0.12)
@@
 		)
 		(fp_line
-			(start -0.261252 -0.735)
-			(end 0.261252 -0.735)
+			(start -0.711252 -1.36)
+			(end 0.711252 -1.36)
 			(stroke
 				(width 0.12)
@@
 		)
 		(fp_rect
-			(start -1.88 -0.98)
-			(end 1.88 0.98)
+			(start -2.48 -1.6)
+			(end 2.48 1.6)
 			(stroke
 				(width 0.05)
@@
 		)
 		(fp_rect
-			(start -1 -0.625)
-			(end 1 0.625)
+			(start -1.6 -1.25)
+			(end 1.6 1.25)
 			(stroke
 				(width 0.1)
@@
 		)
 		(fp_text user "${REFERENCE}"
-			(at 0 0 90)
+			(at 0 0 270)
 			(layer "F.Fab")
 			(effects
 				(font
-					(size 0.5 0.5)
-					(thickness 0.08)
+					(size 0.8 0.8)
+					(thickness 0.12)
 				)
 			)
 		)
 		(pad "1" smd roundrect
-			(at -1.0375 0 270)
-			(size 1.175 1.45)
+			(at -1.5625 0 270)
+			(size 1.325 2.7)
 			(layers "F.Cu" "F.Mask" "F.Paste")
-			(roundrect_rratio 0.212766)
+			(roundrect_rratio 0.188679)
 			(net "/+5V_PI")
 			(pintype "passive")
 		)
 		(pad "2" smd roundrect
-			(at 1.0375 0 270)
-			(size 1.175 1.45)
+			(at 1.5625 0 270)
+			(size 1.325 2.7)
 			(layers "F.Cu" "F.Mask" "F.Paste")
-			(roundrect_rratio 0.212766)
+			(roundrect_rratio 0.188679)
 			(net "/GND")
 			(pintype "passive")
 		)
 		(embedded_fonts no)
-		(model "${KICAD10_3DMODEL_DIR}/Capacitor_SMD.3dshapes/C_0805_2012Metric.step"
+		(model "${KICAD10_3DMODEL_DIR}/Capacitor_SMD.3dshapes/C_1210_3225Metric.step"
 			(offset
 				(xyz 0 0 0)
@@
 	)
 	(segment
-		(start 106.2484 52.4512)
-		(end 107.3296 51.37)
+		(start 106.2484 59.7156)
+		(end 109.3472 59.7156)
 		(width 1)
 		(layer "F.Cu")
@@
 	)
 	(segment
-		(start 112.446 59.7156)
-		(end 109.14 59.7156)
+		(start 108.37 51.37)
+		(end 107.2788 51.37)
 		(width 1)
 		(layer "F.Cu")
@@
 	)
 	(segment
-		(start 107.3296 51.37)
-		(end 108.37 51.37)
+		(start 107.2788 51.37)
+		(end 106.2484 52.4004)
 		(width 1)
 		(layer "F.Cu")
@@
 	)
 	(segment
-		(start 109.14 59.7156)
+		(start 106.2484 52.4004)
 		(end 106.2484 59.7156)
 		(width 1)
@@
 	)
 	(segment
-		(start 106.2484 59.7156)
-		(end 106.2484 52.4512)
+		(start 110.91 51.37)
+		(end 108.37 51.37)
 		(width 1)
 		(layer "F.Cu")
@@
 	)
 	(segment
-		(start 108.37 51.37)
-		(end 110.91 51.37)
+		(start 109.3472 59.7156)
+		(end 112.446 59.7156)
 		(width 1)
 		(layer "F.Cu")

Commit message: Hopefully correct locations.
Parts:
- moved C13 0.40 mm to (123.8, 84.3)
- moved C16 0.40 mm to (110.9, 84.3)
- moved J2 0.40 mm to (114.8, 84.2)
- moved J3 0.40 mm to (127.7, 86.8)
- moved J4 0.40 mm to (107.1, 79.2)
- moved R6 0.40 mm to (131.5, 84.3)
- moved R9 0.40 mm to (103.2, 84.3)
- moved C14 0.40 mm to (123.8, 81.7)
- moved C15 0.40 mm to (110.9, 81.7)
- moved R7 0.40 mm to (131.5, 81.7)
- moved R8 0.40 mm to (103.2, 81.7)
Routing:
- net /+48V_SW: track 56.7 -> 55.6 mm
